File: usb_power2.kicad_pcb (KiCad board)
At the start: 2 copper layers, 31.5 x 21.3 mm, 4 parts, among them J1 USB3_A_Male, J2 Barrel_Jack, J3 USB3_A_SATA_DRIVE, U1 LM7805_TO220

Commit message: Add files via upload
Parts:
- removed U1: LM7805_TO220, Package_TO_SOT_THT:TO-220-3_Vertical
- added R1: 1k, Resistor_THT:R_Axial_DIN0207_L6.3mm_D2.5mm_P2.54mm_Vertical, F.Cu at (99.3, 75.7)
Connections:
- J1 pad 5: SSRX- -> SSTX-
- J1 pad 6: SSRX+ -> SSTX+
- J1 pad 8: SSTX- -> SSRX-
- J1 pad 9: SSTX+ -> SSRX+
- J2 pad 2: Net-(J2-Pad2) -> GND
Routing:
- net Net-(J2-Pad2): track 17.2 -> 0.00 mm
- net GND: track 23.7 -> 33.1 mm, vias 2 -> 1
- net SSTX-: track 5.61 -> 14.7 mm
- net SSTX+: track 5.19 -> 12.4 mm, vias 0 -> 2
- net Net-(J3-Pad1): track 12.0 -> 17.4 mm
- net D-: track 8.53 -> 5.19 mm, vias 2 -> 0
- net SSRX-: track 12.4 -> 15.3 mm, vias 0 -> 2
- net Net-(J2-Pad1): track 8.19 -> 5.45 mm
- net SSRX+: track 11.7 -> 10.8 mm
