File: usb_power2.kicad_sch (KiCad schematic)
At the start: 4 parts, among them J1 USB3_A_Male, J2 Barrel_Jack, J3 USB3_A_SATA_DRIVE, U1 LM7805_TO220

Commit message: Add files via upload
Parts:
- removed U1: LM7805_TO220, Package_TO_SOT_THT:TO-220-3_Vertical, symbol Regulator_Linear:LM7805_TO220
- added R1: 1k, Resistor_THT:R_Axial_DIN0207_L6.3mm_D2.5mm_P2.54mm_Vertical, symbol Device:R_Small_US
- J1: Digikey Part Number (none) -> AE10703-ND
- J3: Digikey Part Number (none) -> AE10704-ND
Connections:
- net GND: now also J2.2
- net SSRX+: now also J1.9 (SSTX+); no longer J1.6 (SSRX+)
- net SSRX-: now also J1.8 (SSTX-); no longer J1.5 (SSRX-)
- net SSTX+: now also J1.6 (SSRX+); no longer J1.9 (SSTX+)
- net SSTX-: now also J1.5 (SSRX-); no longer J1.8 (SSTX-)
- net at J2.1: now also R1.1
- net at J3.1 (VBUS): now also R1.2
Changed lines of the file:
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@@
+    (stroke (width 0) (type default) (color 0 0 0 0))
+  )
+  (wire (pts (xy 91.44 128.27) (xy 107.95 128.27))
     (stroke (width 0) (type default) (color 0 0 0 0))
   )
@@
     (stroke (width 0) (type default) (color 0 0 0 0))
   )
-  (wire (pts (xy 85.09 128.27) (xy 107.95 128.27))
-    (stroke (width 0) (type default) (color 0 0 0 0))
-  )
   (wire (pts (xy 50.8 85.09) (xy 55.88 85.09))
     (stroke (width 0) (type default) (color 0 0 0 0))
@@
     (stroke (width 0) (type default) (color 0 0 0 0))
   )
+  (wire (pts (xy 77.47 157.48) (xy 77.47 161.29))
+    (stroke (width 0) (type default) (color 0 0 0 0))
+  )
   (wire (pts (xy 38.1 92.71) (xy 38.1 97.79))
     (stroke (width 0) (type default) (color 0 0 0 0))
@@
     (stroke (width 0) (type default) (color 0 0 0 0))
   )
+  (wire (pts (xy 69.85 128.27) (xy 86.36 128.27))
+    (stroke (width 0) (type default) (color 0 0 0 0))
+  )
   (wire (pts (xy 111.76 74.93) (xy 118.11 74.93))
     (stroke (width 0) (type default) (color 0 0 0 0))
   )
-  (wire (pts (xy 77.47 135.89) (xy 77.47 161.29))
-    (stroke (width 0) (type default) (color 0 0 0 0))
-  )
   (wire (pts (xy 107.95 128.27) (xy 107.95 87.63))
     (stroke (width 0) (type default) (color 0 0 0 0))
@@
     )
   )
-  (global_label "SSTX+" (shape input) (at 55.88 87.63 0) (fields_autoplaced)
-    (effects (font (size 1.27 1.27)) (justify left))
-    (property "Intersheet References" "${INTERSHEET_REFS}" (id 0) (at 64.4617 87.5506 0)
+  (global_label "SSRX+" (shape input) (at 55.88 87.63 0) (fields_autoplaced)
+    (effects (font (size 1.27 1.27)) (justify left))
+    (property "Intersheet References" "${INTERSHEET_REFS}" (id 0) (at 64.7641 87.5506 0)
       (effects (font (size 1.27 1.27)) (justify left) hide)
     )
@@
     )
   )
-  (global_label "SSTX-" (shape input) (at 55.88 85.09 0) (fields_autoplaced)
-    (effects (font (size 1.27 1.27)) (justify left))
-    (property "Intersheet References" "${INTERSHEET_REFS}" (id 0) (at 64.4617 85.0106 0)
-      (effects (font (size 1.27 1.27)) (justify left) hide)
-    )
-  )
-  (global_label "SSRX-" (shape input) (at 55.88 77.47 0) (fields_autoplaced)
-    (effects (font (size 1.27 1.27)) (justify left))
-    (property "Intersheet References" "${INTERSHEET_REFS}" (id 0) (at 64.7641 77.3906 0)
+  (global_label "SSRX-" (shape input) (at 55.88 85.09 0) (fields_autoplaced)
+    (effects (font (size 1.27 1.27)) (justify left))
+    (property "Intersheet References" "${INTERSHEET_REFS}" (id 0) (at 64.7641 85.0106 0)
+      (effects (font (size 1.27 1.27)) (justify left) hide)
+    )
+  )
+  (global_label "SSTX-" (shape input) (at 55.88 77.47 0) (fields_autoplaced)
+    (effects (font (size 1.27 1.27)) (justify left))
+    (property "Intersheet References" "${INTERSHEET_REFS}" (id 0) (at 64.4617 77.3906 0)
       (effects (font (size 1.27 1.27)) (justify left) hide)
     )
@@
     )
   )
-  (global_label "SSRX+" (shape input) (at 55.88 80.01 0) (fields_autoplaced)
-    (effects (font (size 1.27 1.27)) (justify left))
-    (property "Intersheet References" "${INTERSHEET_REFS}" (id 0) (at 64.7641 79.9306 0)
+  (global_label "SSTX+" (shape input) (at 55.88 80.01 0) (fields_autoplaced)
+    (effects (font (size 1.27 1.27)) (justify left))
+    (property "Intersheet References" "${INTERSHEET_REFS}" (id 0) (at 64.4617 79.9306 0)
       (effects (font (size 1.27 1.27)) (justify left) hide)
     )
@@
     )
     (property "Purchase Link" "https://www.digikey.com/en/products/detail/assmann-wsw-components/AU-Y1006-3/2700523" (id 4) (at 130.81 77.47 0)
+      (effects (font (size 1.27 1.27)) hide)
+    )
+    (property "Digikey Part Number" "AE10704-ND" (id 5) (at 130.81 77.47 0)
       (effects (font (size 1.27 1.27)) hide)
     )
@@
     (pin "9")
   )
+  (symbol (lib_id "power:GND") (at 77.47 157.48 180) (unit 1)
+    (in_bom yes) (on_board yes) (fields_autoplaced)
+    (property "Reference" "#PWR0103" (id 0) (at 77.47 151.13 0)
+      (effects (font (size 1.27 1.27)) hide)
+    )
+    (property "Value" "GND" (id 1) (at 77.47 152.4 0))
+    (property "Footprint" "" (id 2) (at 77.47 157.48 0)
+      (effects (font (size 1.27 1.27)) hide)
+    )
+    (property "Datasheet" "" (id 3) (at 77.47 157.48 0)
+      (effects (font (size 1.27 1.27)) hide)
+    )
+    (pin "1")
+  )
   (symbol (lib_id "power:GND") (at 130.81 54.61 180) (unit 1)
     (in_bom yes) (on_board yes) (fields_autoplaced)
@@
     )
     (property "Datasheet" "~" (id 3) (at 41.91 72.39 0)
+      (effects (font (size 1.27 1.27)) hide)
+    )
+    (property "Digikey Part Number" "AE10703-ND" (id 4) (at 38.1 74.93 0)
       (effects (font (size 1.27 1.27)) hide)
     )
@@
     (pin "9")
   )
-  (symbol (lib_id "Regulator_Linear:LM7805_TO220") (at 77.47 128.27 0) (unit 1)
-    (in_bom yes) (on_board yes) (fields_autoplaced)
-    (property "Reference" "U1" (id 0) (at 77.47 120.65 0))
-    (property "Value" "LM7805_TO220" (id 1) (at 77.47 123.19 0))
-    (property "Footprint" "Package_TO_SOT_THT:TO-220-3_Vertical" (id 2) (at 77.47 122.555 0)
-      (effects (font (size 1.27 1.27) italic) hide)
-    )
-    (property "Datasheet" "https://www.onsemi.cn/PowerSolutions/document/MC7800-D.PDF" (id 3) (at 77.47 129.54 0)
-      (effects (font (size 1.27 1.27)) hide)
-    )
-    (pin "1")
-    (pin "2")
-    (pin "3")
+  (symbol (lib_id "Device:R_Small_US") (at 88.9 128.27 90) (unit 1)
+    (in_bom yes) (on_board yes) (fields_autoplaced)
+    (property "Reference" "R1" (id 0) (at 88.9 121.92 90))
+    (property "Value" "1k" (id 1) (at 88.9 124.46 90))
+    (property "Footprint" "Resistor_THT:R_Axial_DIN0207_L6.3mm_D2.5mm_P2.54mm_Vertical" (id 2) (at 88.9 128.27 0)
+      (effects (font (size 1.27 1.27)) hide)
+    )
+    (property "Datasheet" "~" (id 3) (at 88.9 128.27 0)
+      (effects (font (size 1.27 1.27)) hide)
+    )
+    (pin "1")
+    (pin "2")
   )
   (symbol (lib_id "power:GND") (at 38.1 97.79 0) (unit 1)
@@
       (reference "#PWR0102") (unit 1) (value "GND") (footprint "")
     )
+    (path "/3a430f27-b74d-48b7-ae8b-dea599478e27"
+      (reference "#PWR0103") (unit 1) (value "GND") (footprint "")
+    )
     (path "/7e09a026-923a-435a-8797-95ab554053cc"
       (reference "J1") (unit 1) (value "USB3_A_Male") (footprint "ASSMANN_A-USB3_A-LP-SMT1")
@@
       (reference "J3") (unit 1) (value "USB3_A_SATA_DRIVE") (footprint "CONNUSB09_AU-Y1006-3_14P3X14P25_ASM:AU-Y1006-3")
     )
-    (path "/c8fe50fb-f630-4682-91b0-beb69433add7"
-      (reference "U1") (unit 1) (value "LM7805_TO220") (footprint "Package_TO_SOT_THT:TO-220-3_Vertical")
-    )
-  )
+    (path "/cb3f34be-d070-4936-a388-418b87fea76a"
+      (reference "R1") (unit 1) (value "1k") (footprint "Resistor_THT:R_Axial_DIN0207_L6.3mm_D2.5mm_P2.54mm_Vertical")
+    )
+  )
